File: piano_aid_pcb.sch (KiCad schematic (older format))
At the start: 21 parts

Commit message: Added component labels
Parts:
- gave numbers to parts that had none: 21
Changed lines of the file:
@@
 $EndDescr
 $Comp
-L piano_aid_pcb-rescue:317030213-317030213 U?
+L piano_aid_pcb-rescue:317030213-317030213 U1
 U 1 1 6137BBB1
 P 4650 3700
-F 0 "U?" H 4650 5167 50  0000 C CNN
+F 0 "U1" H 4650 5167 50  0000 C CNN
 F 1 "317030213" H 4650 5076 50  0000 C CNN
 F 2 "XCVR_317030213" H 4650 3700 50  0001 L BNN
@@
 $EndComp
 $Comp
-L Connector:Barrel_Jack_MountingPin J?
+L Connector:Barrel_Jack_MountingPin J1
 U 1 1 613836B9
 P 1100 1000
-F 0 "J?" H 1157 1317 50  0000 C CNN
+F 0 "J1" H 1157 1317 50  0000 C CNN
 F 1 "Barrel_Jack_MountingPin" H 1157 1226 50  0000 C CNN
 F 2 "" H 1150 960 50  0001 C CNN
@@
 $EndComp
 $Comp
-L 74xGxx:74AHCT1G125 U?
+L 74xGxx:74AHCT1G125 U3
 U 1 1 6138B78A
 P 7950 2800
-F 0 "U?" H 7925 2625 50  0000 C CNN
+F 0 "U3" H 7925 2625 50  0000 C CNN
 F 1 "74AHCT1G125" H 7925 2534 50  0000 C CNN
 F 2 "" H 7950 2800 50  0001 C CNN
@@
 $EndComp
 $Comp
-L Device:CP1 C?
+L Device:CP1 C1
 U 1 1 61397A33
 P 1650 1000
-F 0 "C?" H 1765 1046 50  0000 L CNN
+F 0 "C1" H 1765 1046 50  0000 L CNN
 F 1 "1000µ" H 1765 955 50  0000 L CNN
 F 2 "" H 1650 1000 50  0001 C CNN
@@
 $EndComp
 $Comp
-L Device:R R?
+L Device:R R6
 U 1 1 6139F900
 P 8550 2800
-F 0 "R?" V 8343 2800 50  0000 C CNN
+F 0 "R6" V 8343 2800 50  0000 C CNN
 F 1 "440" V 8434 2800 50  0000 C CNN
 F 2 "" V 8480 2800 50  0001 C CNN
@@
 	5650 3700 6900 3700
 $Comp
-L Connector:Conn_01x06_Female J?
+L Connector:Conn_01x06_Female J4
 U 1 1 613D4830
 P 1000 3100
-F 0 "J?" H 892 2575 50  0000 C CNN
+F 0 "J4" H 892 2575 50  0000 C CNN
 F 1 "Conn_01x06_Female" H 892 2666 50  0000 C CNN
 F 2 "" H 1000 3100 50  0001 C CNN
@@
 RESET
 $Comp
-L Device:R R?
+L Device:R R5
 U 1 1 613FD86A
 P 8900 4350
-F 0 "R?" V 8693 4350 50  0000 C CNN
+F 0 "R5" V 8693 4350 50  0000 C CNN
 F 1 "10k" V 8784 4350 50  0000 C CNN
 F 2 "" V 8830 4350 50  0001 C CNN
@@
 	8900 4200 9250 4200
 $Comp
-L Connector:Micro_SD_Card J?
+L Connector:Micro_SD_Card J5
 U 1 1 6139C8E1
 P 10150 4000
-F 0 "J?" H 10100 4717 50  0000 C CNN
+F 0 "J5" H 10100 4717 50  0000 C CNN
 F 1 "Micro_SD_Card" H 10100 4626 50  0000 C CNN
 F 2 "" H 11300 4300 50  0001 C CNN
@@
 	8300 4500 8900 4500
 $Comp
-L Regulator_Linear:AZ1117-3.3 U?
+L Regulator_Linear:AZ1117-3.3 U4
 U 1 1 6144F069
 P 1800 2050
-F 0 "U?" H 1800 2199 50  0000 C CNN
+F 0 "U4" H 1800 2199 50  0000 C CNN
 F 1 "AZ1117-3.3" H 1800 2290 50  0000 C CNN
 F 2 "" H 1800 2300 50  0001 C CIN
@@
 Connection ~ 2100 1150
 $Comp
-L Device:CP1 C?
+L Device:CP1 C4
 U 1 1 61457074
 P 1950 1550
-F 0 "C?" V 1698 1550 50  0000 C CNN
+F 0 "C4" V 1698 1550 50  0000 C CNN
 F 1 "10µ" V 1789 1550 50  0000 C CNN
 F 2 "" H 1950 1550 50  0001 C CNN
@@
 $EndComp
 $Comp
-L Device:CP1 C?
+L Device:CP1 C3
 U 1 1 6145E06D
 P 1650 1550
-F 0 "C?" V 1902 1550 50  0000 C CNN
+F 0 "C3" V 1902 1550 50  0000 C CNN
 F 1 "22µ" V 1811 1550 50  0000 C CNN
 F 2 "" H 1650 1550 50  0001 C CNN
@@
 3.3V
 $Comp
-L Connector:Screw_Terminal_01x02 J?
+L Connector:Screw_Terminal_01x02 J2
 U 1 1 61467FBD
 P 2600 600
-F 0 "J?" V 2564 412 50  0000 R CNN
+F 0 "J2" V 2564 412 50  0000 R CNN
 F 1 "Screw_Terminal_01x02" V 2473 412 50  0000 R CNN
 F 2 "" H 2600 600 50  0001 C CNN
@@
 	1200 3300 2000 3300
 $Comp
-L Device:CP1 C?
+L Device:CP1 C2
 U 1 1 61480AF3
 P 2250 1000
-F 0 "C?" H 2365 1046 50  0000 L CNN
+F 0 "C2" H 2365 1046 50  0000 L CNN
 F 1 "0.1µ" H 2365 955 50  0000 L CNN
 F 2 "" H 2250 1000 50  0001 C CNN
@@
 	1350 6250 1600 6250
 $Comp
-L Connector:DIN-5_180degree J?
+L Connector:DIN-5_180degree J3
 U 1 1 61399AC9
 P 1050 6150
-F 0 "J?" H 1050 5875 50  0000 C CNN
+F 0 "J3" H 1050 5875 50  0000 C CNN
 F 1 "DIN-5_180degree" H 1050 5784 50  0000 C CNN
 F 2 "" H 1050 6150 50  0001 C CNN
@@
 $EndComp
 $Comp
-L Diode:1N914 D?
+L Diode:1N914 D1
 U 1 1 613A3625
 P 2000 6400
-F 0 "D?" V 1954 6479 50  0000 L CNN
+F 0 "D1" V 1954 6479 50  0000 L CNN
 F 1 "1N914" V 2045 6479 50  0000 L CNN
 F 2 "Diode_THT:D_DO-35_SOD27_P7.62mm_Horizontal" H 2000 6225 50  0001 C CNN
@@
 	2300 6550 2300 6500
 $Comp
-L Device:R R?
+L Device:R R3
 U 1 1 61445BFE
 P 3000 6800
-F 0 "R?" H 3070 6846 50  0000 L CNN
+F 0 "R3" H 3070 6846 50  0000 L CNN
 F 1 "4.7k" H 3070 6755 50  0000 L CNN
 F 2 "" V 2930 6800 50  0001 C CNN
@@
 GND
 $Comp
-L Device:CP1 C?
+L Device:CP1 C5
 U 1 1 6148405B
 P 1050 6600
-F 0 "C?" H 1165 6646 50  0000 L CNN
+F 0 "C5" H 1165 6646 50  0000 L CNN
 F 1 "0.1µ" H 1165 6555 50  0000 L CNN
 F 2 "" H 1050 6600 50  0001 C CNN
@@
 GND
 $Comp
-L Device:R R?
+L Device:R R1
 U 1 1 613ABD6D
 P 1750 6250
-F 0 "R?" V 1957 6250 50  0000 C CNN
+F 0 "R1" V 1957 6250 50  0000 C CNN
 F 1 "220" V 1866 6250 50  0000 C CNN
 F 2 "" V 1680 6250 50  0001 C CNN
@@
 NoConn ~ 1500 6150
 $Comp
-L Device:R R?
+L Device:R R2
 U 1 1 614B717D
 P 3250 6250
-F 0 "R?" H 3320 6296 50  0000 L CNN
+F 0 "R2" H 3320 6296 50  0000 L CNN
 F 1 "220" H 3320 6205 50  0000 L CNN
 F 2 "" V 3180 6250 50  0001 C CNN
@@
 $EndComp
 $Comp
-L Isolator:6N138 U?
+L Isolator:6N138 U2
 U 1 1 613CE47C
 P 2600 6400
-F 0 "U?" H 2600 6867 50  0000 C CNN
+F 0 "U2" H 2600 6867 50  0000 C CNN
 F 1 "6N138" H 2600 6776 50  0000 C CNN
 F 2 "" H 2890 6100 50  0001 C CNN
@@
 	8700 4200 8900 4200
 $Comp
-L Device:R R?
+L Device:R R4
 U 1 1 6146BED1
 P 8700 4700
-F 0 "R?" V 8493 4700 50  0000 C CNN
+F 0 "R4" V 8493 4700 50  0000 C CNN
 F 1 "10k" V 8584 4700 50  0000 C CNN
 F 2 "" V 8630 4700 50  0001 C CNN

Commit message: Added LEDs, fixed absolute paths linked to my specific path
Parts:
- added D?: LED_GREEN, symbol Device:LED
- added D?: LED_BLUE, symbol Device:LED
- added R? (x2): 220, symbol Device:R
Connections:
- wire segments 86 -> 94
Changed lines of the file:
@@
 Wire Wire Line
 	8700 4900 8700 4850
+$Comp
+L Device:LED D?
+U 1 1 614AB7E3
+P 2900 4400
+F 0 "D?" V 2939 4282 50  0000 R CNN
+F 1 "LED_GREEN" V 2848 4282 50  0000 R CNN
+F 2 "" H 2900 4400 50  0001 C CNN
+F 3 "~" H 2900 4400 50  0001 C CNN
+	1    2900 4400
+	0    -1   -1   0
+$EndComp
+$Comp
+L Device:LED D?
+U 1 1 614AC0DB
+P 2150 4400
+F 0 "D?" V 2189 4283 50  0000 R CNN
+F 1 "LED_BLUE" V 2098 4283 50  0000 R CNN
+F 2 "" H 2150 4400 50  0001 C CNN
+F 3 "~" H 2150 4400 50  0001 C CNN
+	1    2150 4400
+	0    -1   -1   0
+$EndComp
+Text GLabel 2150 5450 3    50   Input ~ 0
+GND
+Text GLabel 2900 5450 3    50   Input ~ 0
+GND
+Wire Wire Line
+	2150 4850 2150 4550
+Wire Wire Line
+	2150 4250 2150 3800
+Wire Wire Line
+	2150 3800 3650 3800
+Wire Wire Line
+	2900 4250 2900 3900
+Wire Wire Line
+	2900 3900 3650 3900
+$Comp
+L Device:R R?
+U 1 1 614D250F
+P 2150 5000
+F 0 "R?" H 2220 5046 50  0000 L CNN
+F 1 "220" H 2220 4955 50  0000 L CNN
+F 2 "" V 2080 5000 50  0001 C CNN
+F 3 "~" H 2150 5000 50  0001 C CNN
+	1    2150 5000
+	1    0    0    -1
+$EndComp
+$Comp
+L Device:R R?
+U 1 1 614D334B
+P 2900 5000
+F 0 "R?" H 2970 5046 50  0000 L CNN
+F 1 "220" H 2970 4955 50  0000 L CNN
+F 2 "" V 2830 5000 50  0001 C CNN
+F 3 "~" H 2900 5000 50  0001 C CNN
+	1    2900 5000
+	1    0    0    -1
+$EndComp
+Wire Wire Line
+	2900 4850 2900 4550
+Wire Wire Line
+	2900 5150 2900 5450
+Wire Wire Line
+	2150 5150 2150 5450
 $EndSCHEMATC

Commit message: Added refs to components
Parts:
- gave numbers to parts that had none: 4
Changed lines of the file:
@@
 	8700 4900 8700 4850
 $Comp
-L Device:LED D?
+L Device:LED D3
 U 1 1 614AB7E3
 P 2900 4400
-F 0 "D?" V 2939 4282 50  0000 R CNN
+F 0 "D3" V 2939 4282 50  0000 R CNN
 F 1 "LED_GREEN" V 2848 4282 50  0000 R CNN
 F 2 "" H 2900 4400 50  0001 C CNN
@@
 $EndComp
 $Comp
-L Device:LED D?
+L Device:LED D2
 U 1 1 614AC0DB
 P 2150 4400
-F 0 "D?" V 2189 4283 50  0000 R CNN
+F 0 "D2" V 2189 4283 50  0000 R CNN
 F 1 "LED_BLUE" V 2098 4283 50  0000 R CNN
 F 2 "" H 2150 4400 50  0001 C CNN
@@
 	2900 3900 3650 3900
 $Comp
-L Device:R R?
+L Device:R R7
 U 1 1 614D250F
 P 2150 5000
-F 0 "R?" H 2220 5046 50  0000 L CNN
+F 0 "R7" H 2220 5046 50  0000 L CNN
 F 1 "220" H 2220 4955 50  0000 L CNN
 F 2 "" V 2080 5000 50  0001 C CNN
@@
 $EndComp
 $Comp
-L Device:R R?
+L Device:R R8
 U 1 1 614D334B
 P 2900 5000
-F 0 "R?" H 2970 5046 50  0000 L CNN
+F 0 "R8" H 2970 5046 50  0000 L CNN
 F 1 "220" H 2970 4955 50  0000 L CNN
 F 2 "" V 2830 5000 50  0001 C CNN

Commit message: Added kicad libraries from adafruit and digkey
Parts:
- removed J2: Screw_Terminal_01x02, symbol Connector:Screw_Terminal_01x02
- added J2: Screw_Terminal_01x03, symbol Connector:Screw_Terminal_01x03
Connections:
- wire segments 94 -> 96
- no-connect marks 3 -> 30
Other:
- moved on the sheet: C1, C2, C3, C4, J1, U4
Changed lines of the file:
@@
 L Connector:Barrel_Jack_MountingPin J1
 U 1 1 613836B9
-P 1100 1000
-F 0 "J1" H 1157 1317 50  0000 C CNN
-F 1 "Barrel_Jack_MountingPin" H 1157 1226 50  0000 C CNN
-F 2 "" H 1150 960 50  0001 C CNN
-F 3 "~" H 1150 960 50  0001 C CNN
-	1    1100 1000
+P 1000 1150
+F 0 "J1" H 1057 1467 50  0000 C CNN
+F 1 "Barrel_Jack_MountingPin" H 1057 1376 50  0000 C CNN
+F 2 "" H 1050 1110 50  0001 C CNN
+F 3 "~" H 1050 1110 50  0001 C CNN
+	1    1000 1150
 	1    0    0    -1
 $EndComp
@@
 L Device:CP1 C1
 U 1 1 61397A33
-P 1650 1000
-F 0 "C1" H 1765 1046 50  0000 L CNN
-F 1 "1000µ" H 1765 955 50  0000 L CNN
-F 2 "" H 1650 1000 50  0001 C CNN
-F 3 "~" H 1650 1000 50  0001 C CNN
-	1    1650 1000
+P 1550 1150
+F 0 "C1" H 1665 1196 50  0000 L CNN
+F 1 "1000µ" H 1665 1105 50  0000 L CNN
+F 2 "" H 1550 1150 50  0001 C CNN
+F 3 "~" H 1550 1150 50  0001 C CNN
+	1    1550 1150
 	1    0    0    -1
 $EndComp
@@
 $EndComp
 Wire Wire Line
-	1400 900  1500 900
-Wire Wire Line
-	1500 900  1500 850
-Wire Wire Line
-	1500 850  1650 850
-Wire Wire Line
-	1400 1100 1500 1100
-Wire Wire Line
-	1500 1100 1500 1150
-Wire Wire Line
-	1500 1150 1650 1150
+	1300 1050 1400 1050
+Wire Wire Line
+	1400 1050 1400 1000
+Wire Wire Line
+	1400 1000 1550 1000
+Wire Wire Line
+	1300 1250 1400 1250
+Wire Wire Line
+	1400 1250 1400 1300
+Wire Wire Line
+	1400 1300 1550 1300
 Wire Wire Line
 	1200 2900 3650 2900
@@
 Wire Wire Line
 	1200 3100 2000 3100
-Text GLabel 3000 850  2    50   Input ~ 0
+Text GLabel 2900 1000 2    50   Input ~ 0
 5V
-Text GLabel 3000 1150 2    50   Input ~ 0
-GND
-Connection ~ 1650 1150
-Connection ~ 1650 850
+Text GLabel 2900 1300 2    50   Input ~ 0
+GND
+Connection ~ 1550 1300
+Connection ~ 1550 1000
 Text GLabel 8650 4200 0    50   Input ~ 0
 3.3V
@@
 L Regulator_Linear:AZ1117-3.3 U4
 U 1 1 6144F069
-P 1800 2050
-F 0 "U4" H 1800 2199 50  0000 C CNN
-F 1 "AZ1117-3.3" H 1800 2290 50  0000 C CNN
-F 2 "" H 1800 2300 50  0001 C CIN
-F 3 "https://www.diodes.com/assets/Datasheets/AZ1117.pdf" H 1800 2050 50  0001 C CNN
-	1    1800 2050
+P 1700 2200
+F 0 "U4" H 1700 2349 50  0000 C CNN
+F 1 "AZ1117-3.3" H 1700 2440 50  0000 C CNN
+F 2 "" H 1700 2450 50  0001 C CIN
+F 3 "https://www.diodes.com/assets/Datasheets/AZ1117.pdf" H 1700 2200 50  0001 C CNN
+	1    1700 2200
 	-1   0    0    1
 $EndComp
 Wire Wire Line
-	1650 1150 1800 1150
-Connection ~ 1800 1150
-Wire Wire Line
-	1800 1150 2100 1150
-Connection ~ 2100 1150
+	1550 1300 1700 1300
+Connection ~ 1700 1300
+Wire Wire Line
+	1700 1300 2000 1300
+Connection ~ 2000 1300
 $Comp
 L Device:CP1 C4
 U 1 1 61457074
-P 1950 1550
-F 0 "C4" V 1698 1550 50  0000 C CNN
-F 1 "10µ" V 1789 1550 50  0000 C CNN
-F 2 "" H 1950 1550 50  0001 C CNN
-F 3 "~" H 1950 1550 50  0001 C CNN
-	1    1950 1550
+P 1850 1700
+F 0 "C4" V 1598 1700 50  0000 C CNN
+F 1 "10µ" V 1689 1700 50  0000 C CNN
+F 2 "" H 1850 1700 50  0001 C CNN
+F 3 "~" H 1850 1700 50  0001 C CNN
+	1    1850 1700
 	0    1    1    0
 $EndComp
@@
 L Device:CP1 C3
 U 1 1 6145E06D
-P 1650 1550
-F 0 "C3" V 1902 1550 50  0000 C CNN
-F 1 "22µ" V 1811 1550 50  0000 C CNN
-F 2 "" H 1650 1550 50  0001 C CNN
-F 3 "~" H 1650 1550 50  0001 C CNN
-	1    1650 1550
+P 1550 1700
+F 0 "C3" V 1802 1700 50  0000 C CNN
+F 1 "22µ" V 1711 1700 50  0000 C CNN
+F 2 "" H 1550 1700 50  0001 C CNN
+F 3 "~" H 1550 1700 50  0001 C CNN
+	1    1550 1700
 	0    -1   -1   0
 $EndComp
-Connection ~ 2100 1550
-Wire Wire Line
-	2100 1550 2100 2050
-Connection ~ 1800 1550
-Wire Wire Line
-	1800 1550 1800 1750
-Wire Wire Line
-	1500 1550 1500 2050
-Wire Wire Line
-	2100 1150 2100 1550
-Wire Wire Line
-	1800 1150 1800 1550
-Wire Wire Line
-	1500 1550 1200 1550
-Connection ~ 1500 1550
-Text GLabel 1200 1550 0    50   Input ~ 0
+Connection ~ 2000 1700
+Wire Wire Line
+	2000 1700 2000 2200
+Connection ~ 1700 1700
+Wire Wire Line
+	1700 1700 1700 1900
+Wire Wire Line
+	1400 1700 1400 2200
+Wire Wire Line
+	2000 1300 2000 1700
+Wire Wire Line
+	1700 1300 1700 1700
+Wire Wire Line
+	1400 1700 1100 1700
+Connection ~ 1400 1700
+Text GLabel 1100 1700 0    50   Input ~ 0
 3.3V
-$Comp
-L Connector:Screw_Terminal_01x02 J2
-U 1 1 61467FBD
-P 2600 600
-F 0 "J2" V 2564 412 50  0000 R CNN
-F 1 "Screw_Terminal_01x02" V 2473 412 50  0000 R CNN
-F 2 "" H 2600 600 50  0001 C CNN
-F 3 "~" H 2600 600 50  0001 C CNN
-	1    2600 600
-	0    -1   -1   0
-$EndComp
-Wire Wire Line
-	2600 850  2600 800
-Wire Wire Line
-	1650 850  2250 850
-Wire Wire Line
-	2600 850  3000 850
-Connection ~ 2600 850
-Wire Wire Line
-	2700 800  2700 1150
-Wire Wire Line
-	2700 1150 3000 1150
-Wire Wire Line
-	2100 1150 2250 1150
-Connection ~ 2700 1150
+Wire Wire Line
+	1550 1000 2150 1000
+Wire Wire Line
+	2500 1000 2900 1000
+Connection ~ 2500 1000
+Wire Wire Line
+	2600 1300 2900 1300
+Wire Wire Line
+	2000 1300 2150 1300
+Connection ~ 2600 1300
 Wire Wire Line
 	7950 2600 7950 2400
@@
 L Device:CP1 C2
 U 1 1 61480AF3
-P 2250 1000
-F 0 "C2" H 2365 1046 50  0000 L CNN
-F 1 "0.1µ" H 2365 955 50  0000 L CNN
-F 2 "" H 2250 1000 50  0001 C CNN
-F 3 "~" H 2250 1000 50  0001 C CNN
-	1    2250 1000
-	1    0    0    -1
-$EndComp
-Connection ~ 2250 850
-Wire Wire Line
-	2250 850  2600 850
-Connection ~ 2250 1150
-Wire Wire Line
-	2250 1150 2700 1150
+P 2150 1150
+F 0 "C2" H 2265 1196 50  0000 L CNN
+F 1 "0.1µ" H 2265 1105 50  0000 L CNN
+F 2 "" H 2150 1150 50  0001 C CNN
+F 3 "~" H 2150 1150 50  0001 C CNN
+	1    2150 1150
+	1    0    0    -1
+$EndComp
+Connection ~ 2150 1000
+Wire Wire Line
+	2150 1000 2500 1000
+Connection ~ 2150 1300
+Wire Wire Line
+	2150 1300 2600 1300
 Wire Wire Line
 	8000 2850 8000 2950
@@
 Wire Wire Line
 	2150 5150 2150 5450
+$Comp
+L Connector:Screw_Terminal_01x03 J2
+U 1 1 614FB8AE
+P 2600 550
+F 0 "J2" V 2564 362 50  0000 R CNN
+F 1 "Screw_Terminal_01x03" V 2473 362 50  0000 R CNN
+F 2 "" H 2600 550 50  0001 C CNN
+F 3 "~" H 2600 550 50  0001 C CNN
+	1    2600 550
+	0    -1   -1   0
+$EndComp
+Wire Wire Line
+	2600 750  2600 1300
+Wire Wire Line
+	2500 750  2500 1000
+Wire Wire Line
+	2700 750  2700 850
+Text GLabel 2900 850  2    50   Input ~ 0
+LED_CONTROL_OUT
+Wire Wire Line
+	2700 850  2900 850
+NoConn ~ 5650 3200
+NoConn ~ 5650 3400
+NoConn ~ 5650 3500
+NoConn ~ 5650 3600
+NoConn ~ 5650 4200
+NoConn ~ 5650 4300
+NoConn ~ 5650 4400
+NoConn ~ 5650 4500
+NoConn ~ 5650 4600
+NoConn ~ 5650 4700
+NoConn ~ 3650 4700
+NoConn ~ 3650 4600
+NoConn ~ 3650 4500
+NoConn ~ 3650 4400
+NoConn ~ 3650 4300
+NoConn ~ 3650 4200
+NoConn ~ 3650 4100
+NoConn ~ 3650 3700
+NoConn ~ 3650 3600
+NoConn ~ 3650 3500
+NoConn ~ 3650 3400
+NoConn ~ 3650 3300
+NoConn ~ 3650 3200
+NoConn ~ 1000 1450
+NoConn ~ 5650 2700
+NoConn ~ 5650 2600
+NoConn ~ 10950 4600
 $EndSCHEMATC
