File: piano_aid_pcb.sch (KiCad schematic (older format))
At the start: 25 parts, among them J1 Barrel_Jack_MountingPin, J2 Screw_Terminal_01x03, J3 DIN-5_180degree, J4 Conn_01x06_Female, J5 Micro_SD_Card, U1 317030213, U2 6N138, U3 74AHCT1G125, U4 AZ1117-3.3

Commit message: Added adafruit eagle libraries. Also Started assigning components to footprints
Parts:
- removed D2: LED_BLUE, symbol Device:LED
- removed D3: LED_GREEN, symbol Device:LED
- removed U3: 74AHCT1G125, symbol 74xGxx:74AHCT1G125
- added D2: LED_BLUE, digikey-footprints:0603, symbol dk_LED-Indication-Discrete:LTST-C191TBKT
- added D3: LED_GREEN, digikey-footprints:0603, symbol dk_LED-Indication-Discrete:LG_L29K-G2J1-24-Z
- added U3: 74AHCT1G125SE-7, 74AHCT1G125SE-7:SOT65P210X110-5N, symbol 74AHCT1G125SE-7:74AHCT1G125SE-7
- J1: footprint (none) -> Connector_BarrelJack:BarrelJack_Horizontal
- J2: footprint (none) -> TerminalBlock:TerminalBlock_bornier-3_P5.08mm
- J3: footprint (none) -> 57PC5F:57PC5F
- J5: footprint (none) -> adafruit:MICROSD
- R1, R2, R3, R4, R5, R6, R7, R8: footprint (none) -> Resistor_SMD:R_0805_2012Metric_Pad1.15x1.40mm_HandSolder
- U1: footprint XCVR_317030213 -> micro:XCVR_317030213
- U4: footprint (none) -> 2021-09-23_22-23-04:AZ1117IH-3.3TRG1
Connections:
- wire segments 96 -> 95
Other:
- moved on the sheet: R6
Changed lines of the file:
@@
 F 0 "U1" H 4650 5167 50  0000 C CNN
 F 1 "317030213" H 4650 5076 50  0000 C CNN
-F 2 "XCVR_317030213" H 4650 3700 50  0001 L BNN
+F 2 "micro:XCVR_317030213" H 4650 3700 50  0001 L BNN
 F 3 "" H 4650 3700 50  0001 L BNN
 F 4 "Manufacturer Recommendations" H 4650 3700 50  0001 L BNN "STANDARD"
@@
 F 0 "J1" H 1057 1467 50  0000 C CNN
 F 1 "Barrel_Jack_MountingPin" H 1057 1376 50  0000 C CNN
-F 2 "" H 1050 1110 50  0001 C CNN
+F 2 "Connector_BarrelJack:BarrelJack_Horizontal" H 1050 1110 50  0001 C CNN
 F 3 "~" H 1050 1110 50  0001 C CNN
 	1    1000 1150
-	1    0    0    -1
-$EndComp
-$Comp
-L 74xGxx:74AHCT1G125 U3
-U 1 1 6138B78A
-P 7950 2800
-F 0 "U3" H 7925 2625 50  0000 C CNN
-F 1 "74AHCT1G125" H 7925 2534 50  0000 C CNN
-F 2 "" H 7950 2800 50  0001 C CNN
-F 3 "http://www.ti.com/lit/sg/scyt129e/scyt129e.pdf" H 7950 2800 50  0001 C CNN
-	1    7950 2800
 	1    0    0    -1
 $EndComp
@@
 L Device:R R6
 U 1 1 6139F900
-P 8550 2800
-F 0 "R6" V 8343 2800 50  0000 C CNN
-F 1 "440" V 8434 2800 50  0000 C CNN
-F 2 "" V 8480 2800 50  0001 C CNN
-F 3 "~" H 8550 2800 50  0001 C CNN
-	1    8550 2800
+P 9400 2500
+F 0 "R6" V 9193 2500 50  0000 C CNN
+F 1 "440" V 9284 2500 50  0000 C CNN
+F 2 "Resistor_SMD:R_0805_2012Metric_Pad1.15x1.40mm_HandSolder" V 9330 2500 50  0001 C CNN
+F 3 "~" H 9400 2500 50  0001 C CNN
+	1    9400 2500
 	0    1    1    0
 $EndComp
@@
 F 0 "R5" V 8693 4350 50  0000 C CNN
 F 1 "10k" V 8784 4350 50  0000 C CNN
-F 2 "" V 8830 4350 50  0001 C CNN
+F 2 "Resistor_SMD:R_0805_2012Metric_Pad1.15x1.40mm_HandSolder" V 8830 4350 50  0001 C CNN
 F 3 "~" H 8900 4350 50  0001 C CNN
 	1    8900 4350
@@
 F 0 "J5" H 10100 4717 50  0000 C CNN
 F 1 "Micro_SD_Card" H 10100 4626 50  0000 C CNN
-F 2 "" H 11300 4300 50  0001 C CNN
+F 2 "adafruit:MICROSD" H 11300 4300 50  0001 C CNN
 F 3 "http://katalog.we-online.de/em/datasheet/693072010801.pdf" H 10150 4000 50  0001 C CNN
 	1    10150 4000
@@
 F 0 "U4" H 1700 2349 50  0000 C CNN
 F 1 "AZ1117-3.3" H 1700 2440 50  0000 C CNN
-F 2 "" H 1700 2450 50  0001 C CIN
+F 2 "2021-09-23_22-23-04:AZ1117IH-3.3TRG1" H 1700 2450 50  0001 C CIN
 F 3 "https://www.diodes.com/assets/Datasheets/AZ1117.pdf" H 1700 2200 50  0001 C CNN
 	1    1700 2200
@@
 Connection ~ 2600 1300
 Wire Wire Line
-	7950 2600 7950 2400
-Wire Wire Line
 	5650 3300 6900 3300
 Wire Wire Line
@@
 	6900 2800 7650 2800
 Wire Wire Line
-	8200 2800 8400 2800
-Wire Wire Line
-	8700 2800 9250 2800
-Text GLabel 9250 2800 2    50   Input ~ 0
+	9050 2500 9250 2500
+Wire Wire Line
+	9550 2500 10100 2500
+Text GLabel 10100 2500 2    50   Input ~ 0
 LED_CONTROL_OUT
 Text GLabel 6900 3700 2    50   Input ~ 0
@@
 Wire Wire Line
 	2150 1300 2600 1300
-Wire Wire Line
-	8000 2850 8000 2950
-Wire Wire Line
-	8000 2950 8300 2950
-Wire Wire Line
-	8300 2950 8300 3250
-Wire Wire Line
-	8000 2750 8000 2650
-Wire Wire Line
-	8000 2650 8300 2650
-Wire Wire Line
-	8300 2650 8300 2400
-Text GLabel 8300 3250 3    50   Input ~ 0
-GND
-Text GLabel 8300 2400 1    50   Input ~ 0
-5V
-Text GLabel 7950 2400 1    50   Input ~ 0
+Text GLabel 7250 3150 3    50   Input ~ 0
 GND
 Wire Wire Line
@@
 F 0 "J3" H 1050 5875 50  0000 C CNN
 F 1 "DIN-5_180degree" H 1050 5784 50  0000 C CNN
-F 2 "" H 1050 6150 50  0001 C CNN
+F 2 "57PC5F:57PC5F" H 1050 6150 50  0001 C CNN
 F 3 "http://www.mouser.com/ds/2/18/40_c091_abd_e-75918.pdf" H 1050 6150 50  0001 C CNN
 	1    1050 6150
@@
 F 0 "R3" H 3070 6846 50  0000 L CNN
 F 1 "4.7k" H 3070 6755 50  0000 L CNN
-F 2 "" V 2930 6800 50  0001 C CNN
+F 2 "Resistor_SMD:R_0805_2012Metric_Pad1.15x1.40mm_HandSolder" V 2930 6800 50  0001 C CNN
 F 3 "~" H 3000 6800 50  0001 C CNN
 	1    3000 6800
@@
 F 0 "R1" V 1957 6250 50  0000 C CNN
 F 1 "220" V 1866 6250 50  0000 C CNN
-F 2 "" V 1680 6250 50  0001 C CNN
+F 2 "Resistor_SMD:R_0805_2012Metric_Pad1.15x1.40mm_HandSolder" V 1680 6250 50  0001 C CNN
 F 3 "~" H 1750 6250 50  0001 C CNN
 	1    1750 6250
@@
 F 0 "R2" H 3320 6296 50  0000 L CNN
 F 1 "220" H 3320 6205 50  0000 L CNN
-F 2 "" V 3180 6250 50  0001 C CNN
+F 2 "Resistor_SMD:R_0805_2012Metric_Pad1.15x1.40mm_HandSolder" V 3180 6250 50  0001 C CNN
 F 3 "~" H 3250 6250 50  0001 C CNN
 	1    3250 6250
@@
 F 0 "R4" V 8493 4700 50  0000 C CNN
 F 1 "10k" V 8584 4700 50  0000 C CNN
-F 2 "" V 8630 4700 50  0001 C CNN
+F 2 "Resistor_SMD:R_0805_2012Metric_Pad1.15x1.40mm_HandSolder" V 8630 4700 50  0001 C CNN
 F 3 "~" H 8700 4700 50  0001 C CNN
 	1    8700 4700
@@
 Wire Wire Line
 	8700 4900 8700 4850
-$Comp
-L Device:LED D3
-U 1 1 614AB7E3
-P 2900 4400
-F 0 "D3" V 2939 4282 50  0000 R CNN
-F 1 "LED_GREEN" V 2848 4282 50  0000 R CNN
-F 2 "" H 2900 4400 50  0001 C CNN
-F 3 "~" H 2900 4400 50  0001 C CNN
-	1    2900 4400
-	0    -1   -1   0
-$EndComp
-$Comp
-L Device:LED D2
-U 1 1 614AC0DB
-P 2150 4400
-F 0 "D2" V 2189 4283 50  0000 R CNN
-F 1 "LED_BLUE" V 2098 4283 50  0000 R CNN
-F 2 "" H 2150 4400 50  0001 C CNN
-F 3 "~" H 2150 4400 50  0001 C CNN
-	1    2150 4400
-	0    -1   -1   0
-$EndComp
 Text GLabel 2150 5450 3    50   Input ~ 0
 GND
@@
 F 0 "R7" H 2220 5046 50  0000 L CNN
 F 1 "220" H 2220 4955 50  0000 L CNN
-F 2 "" V 2080 5000 50  0001 C CNN
+F 2 "Resistor_SMD:R_0805_2012Metric_Pad1.15x1.40mm_HandSolder" V 2080 5000 50  0001 C CNN
 F 3 "~" H 2150 5000 50  0001 C CNN
 	1    2150 5000
@@
 F 0 "R8" H 2970 5046 50  0000 L CNN
 F 1 "220" H 2970 4955 50  0000 L CNN
-F 2 "" V 2830 5000 50  0001 C CNN
+F 2 "Resistor_SMD:R_0805_2012Metric_Pad1.15x1.40mm_HandSolder" V 2830 5000 50  0001 C CNN
 F 3 "~" H 2900 5000 50  0001 C CNN
 	1    2900 5000
@@
 F 0 "J2" V 2564 362 50  0000 R CNN
 F 1 "Screw_Terminal_01x03" V 2473 362 50  0000 R CNN
-F 2 "" H 2600 550 50  0001 C CNN
+F 2 "TerminalBlock:TerminalBlock_bornier-3_P5.08mm" H 2600 550 50  0001 C CNN
 F 3 "~" H 2600 550 50  0001 C CNN
 	1    2600 550
@@
 NoConn ~ 5650 2600
 NoConn ~ 10950 4600
+$Comp
+L 74AHCT1G125SE-7:74AHCT1G125SE-7 U3
+U 1 1 614DDF7F
+P 8350 2600
+F 0 "U3" H 8350 3070 50  0000 C CNN
+F 1 "74AHCT1G125SE-7" H 8350 2979 50  0000 C CNN
+F 2 "74AHCT1G125SE-7:SOT65P210X110-5N" H 8350 2600 50  0001 L BNN
+F 3 "" H 8350 2600 50  0001 L BNN
+F 4 "Diodes INC" H 8350 2600 50  0001 L BNN "SUPPLIER"
+F 5 "SOT-353-5" H 8350 2600 50  0001 L BNN "PACKAGE"
+F 6 "64T4871" H 8350 2600 50  0001 L BNN "OC_NEWARK"
+F 7 "2057391" H 8350 2600 50  0001 L BNN "OC_FARNELL"
+F 8 "74AHCT1G125SE-7" H 8350 2600 50  0001 L BNN "MPN"
+	1    8350 2600
+	1    0    0    -1
+$EndComp
+Wire Wire Line
+	7650 2700 7250 2700
+Wire Wire Line
+	7250 2500 7650 2500
+Wire Wire Line
+	7250 2500 7250 2250
+Wire Wire Line
+	7250 3150 7250 3000
+Wire Wire Line
+	7250 3000 7650 3000
+Wire Wire Line
+	7250 2700 7250 3000
+Connection ~ 7250 3000
+Text GLabel 7250 2250 1    50   Input ~ 0
+5V
+$Comp
+L dk_LED-Indication-Discrete:LTST-C191TBKT D2
+U 1 1 61506421
+P 2150 4450
+F 0 "D2" V 2047 4628 60  0000 L CNN
+F 1 "LED_BLUE" V 2153 4628 60  0000 L CNN
+F 2 "digikey-footprints:0603" H 2350 4650 60  0001 L CNN
+F 3 "http://optoelectronics.liteon.com/upload/download/DS22-2000-230/LTST-C191TBKT.pdf" H 2350 4750 60  0001 L CNN
+F 4 "160-1647-1-ND" H 2350 4850 60  0001 L CNN "Digi-Key_PN"
+F 5 "LTST-C191TBKT" H 2350 4950 60  0001 L CNN "MPN"
+F 6 "Optoelectronics" H 2350 5050 60  0001 L CNN "Category"
+F 7 "LED Indication - Discrete" H 2350 5150 60  0001 L CNN "Family"
+F 8 "http://optoelectronics.liteon.com/upload/download/DS22-2000-230/LTST-C191TBKT.pdf" H 2350 5250 60  0001 L CNN "DK_Datasheet_Link"
+F 9 "/product-detail/en/lite-on-inc/LTST-C191TBKT/160-1647-1-ND/573587" H 2350 5350 60  0001 L CNN "DK_Detail_Page"
+F 10 "LED BLUE CLEAR CHIP SMD" H 2350 5450 60  0001 L CNN "Description"
+F 11 "Lite-On Inc." H 2350 5550 60  0001 L CNN "Manufacturer"
+F 12 "Active" H 2350 5650 60  0001 L CNN "Status"
+	1    2150 4450
+	0    1    1    0
+$EndComp
+$Comp
+L dk_LED-Indication-Discrete:LG_L29K-G2J1-24-Z D3
+U 1 1 615118D7
+P 2900 4450
+F 0 "D3" V 2797 4628 60  0000 L CNN
+F 1 "LED_GREEN" V 2903 4628 60  0000 L CNN
+F 2 "digikey-footprints:0603" H 3100 4650 60  0001 L CNN
+F 3 "https://dammedia.osram.info/media/resource/hires/osram-dam-2493945/LG%20L29K.pdf" H 3100 4750 60  0001 L CNN
+F 4 "475-2709-1-ND" H 3100 4850 60  0001 L CNN "Digi-Key_PN"
+F 5 "LG L29K-G2J1-24-Z" H 3100 4950 60  0001 L CNN "MPN"
+F 6 "Optoelectronics" H 3100 5050 60  0001 L CNN "Category"
+F 7 "LED Indication - Discrete" H 3100 5150 60  0001 L CNN "Family"
+F 8 "https://dammedia.osram.info/media/resource/hires/osram-dam-2493945/LG%20L29K.pdf" H 3100 5250 60  0001 L CNN "DK_Datasheet_Link"
+F 9 "/product-detail/en/osram-opto-semiconductors-inc/LG-L29K-G2J1-24-Z/475-2709-1-ND/1938876" H 3100 5350 60  0001 L CNN "DK_Detail_Page"
+F 10 "LED GREEN DIFFUSED 0603 SMD" H 3100 5450 60  0001 L CNN "Description"
+F 11 "OSRAM Opto Semiconductors Inc." H 3100 5550 60  0001 L CNN "Manufacturer"
+F 12 "Active" H 3100 5650 60  0001 L CNN "Status"
+	1    2900 4450
+	0    1    1    0
+$EndComp
 $EndSCHEMATC
