File: piano_aid_pcb.kicad_pcb (KiCad board)
At the start: 2 copper layers, 44.5 x 61 mm, 37 parts, among them J1 PJ-082BH, J2 796644-3, J3 DIN-5_180degree, J4 Conn_01x06_Female, J5 Micro_SD_Card_Det, J6 Conn_01x07_Female, U1 317030213, U2 6N138, U3 74AHCT1G125W5-7, U4 AZ1117-3.3

Commit message: Made schematic a bit neater
Other:
- board text added: "S/N"
Changed lines of the file:
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@@
   (general
     (thickness 1.6)
-    (drawings 26)
+    (drawings 28)
     (tracks 337)
     (zones 0)
@@
   (page A4)
   (title_block
-    (title "P.I.A.N.O PCB")
-    (date 2021-09-24)
-    (rev v02)
-    (comment 4 "Authors: Jared Botte, Jerry Jin")
+    (title P.I.A.N.O)
+    (date 2021-10-06)
+    (rev 2)
+    (comment 3 "Tong Wang, Kirk Weibel")
+    (comment 4 "Authors: Jared Botte, Jerry Liu")
   )
   (layers
@@
   )
   (setup
-    (last_trace_width 0.635)
+    (last_trace_width 0.1524)
     (user_trace_width 0.3048)
     (user_trace_width 0.635)
@@
     )
   )
+  (gr_text S/N (at 134.366 132.588) (layer B.SilkS)
+    (effects (font (size 1 1) (thickness 0.15)) (justify mirror))
+  )
+  (gr_poly (pts (xy 136.652 131.572) (xy 131.572 131.572) (xy 131.572 127.254) (xy 136.652 127.254)) (layer B.SilkS) (width 0.1))
   (gr_arc (start 123.19 132.08) (end 120.65 132.08) (angle -90) (layer Edge.Cuts) (width 0.05))
   (gr_arc (start 162.56 132.08) (end 162.56 134.62) (angle -90) (layer Edge.Cuts) (width 0.05))

Commit message: Fixed keepout zone, cleaned traces
Routing:
- net CLK: track 61.1 -> 59.7 mm, vias 1 -> 0
- net CMD: track 59.2 -> 58.0 mm
- net DAT0: track 64.4 -> 63.2 mm, vias 3 -> 2
